File: PCB/SlantPad.kicad_pcb (KiCad board)
At the start: 2 copper layers, 67.1 x 67.5 mm, 37 parts, among them SW1 SW_Push, SW10 RotaryEncoder_Switch, SW2 SW_Push, SW3 SW_Push, SW4 SW_Push, SW5 SW_Push, SW6 SW_Push, SW7 SW_Push, SW8 SW_Push, SW9 SW_Push, U1 XIAO-RP2040-DIP

Commit message: updated README.md
Other:
- board text added: "SlantPad be like"
- board text removed: "CADPad"
